File: ADSR-Panel.kicad_pcb (KiCad board)
At the start: 2 copper layers, 10 x 128.5 mm, 17 parts

Commit message: Finished panel
Parts:
- added ~: ~, KraakenStuff_ADSR:Panel_Graphics_ADSR_Out, F.Cu at (4.95, 109.1)
- added ~: ~, KraakenStuff_ADSR:Panel_Graphics_ADSR_GateIn, F.Cu at (5.08, 97.3)
- ~: value LOGO -> ~
- ~ (x2): value Panel_Screw_Elliptical -> ~
- ~: value Panel_Screw_Hole_2.6mm -> ~
- ~ (x2): value Panel_Thonkiconn_6mm -> ~
- ~ (x2): value Panel_Trimmer_6.7mm -> ~
- ~: footprint KraakenStuff:Kraakenstuff_2HP -> KraakenStuff:Kraakenstuff_15mm
Other:
- board text removed: "It's hand made, bro! And there are only five of them in the known universe."
- board text removed: "The price he's asking for this module is at least a quarter of what it's really worth."
- board text removed: "This death metal edition of ADSR, dedicated to Paul Bergel, is extremely rare."
